File: electronics/sensor-epaper/sensor-epaper.kicad_sch (KiCad schematic)
At the start: 88 parts, among them J1 i2c, J2 Conn_01x06, J3 Ufl, J4 Display, J9 USB micro, Q1 Q_NMOS_GSD, Q3 NX2301P, SW1 SW_Push, U1 ESP32-C3FN4, U2 AMS1117-3.3, U3 NCP1421, U4 SHT40-AD1B-R2, Y2 32kHz, Y3 40MHz 10ppm

Commit message: Add missed electronics files for PCB 1.2.0
Parts:
- removed C48: 1u, Capacitor_SMD:C_0402_1005Metric, symbol Device:C
- C43, C44: value 1u -> 4u7; LCSC C52923 -> C19666
Changed lines of the file:
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@@
-(kicad_sch (version 20221110) (generator eeschema)
+(kicad_sch (version 20221004) (generator eeschema)
   (paper "A3")
   (title_block
@@
   (junction (at 91.44 62.23) (diameter 0) (color 0 0 0 0)
   )
-  (junction (at 388.62 234.95) (diameter 0) (color 0 0 0 0)
-  )
   (junction (at 372.11 38.735) (diameter 0) (color 0 0 0 0)
   )
   (junction (at 279.4 163.83) (diameter 0) (color 0 0 0 0)
   )
-  (junction (at 388.62 245.11) (diameter 0) (color 0 0 0 0)
-  )
   (junction (at 119.38 24.765) (diameter 0) (color 0 0 0 0)
   )
@@
     (stroke (width 0) (type default))
   )
-  (wire (pts (xy 388.62 242.57) (xy 388.62 245.11))
-    (stroke (width 0) (type default))
-  )
   (wire (pts (xy 153.67 46.99) (xy 153.67 48.26))
     (stroke (width 0) (type default))
@@
     )
   )
-  (symbol (lib_id "Device:C") (at 388.62 238.76 0) (unit 1)
-    (in_bom yes) (on_board yes) (dnp no)
-    (property "Reference" "C48" (at 391.541 237.5916 0)
-      (effects (font (size 1.27 1.27)) (justify left))
-    )
-    (property "Value" "1u" (at 391.541 239.903 0)
-      (effects (font (size 1.27 1.27)) (justify left))
-    )
-    (property "Footprint" "Capacitor_SMD:C_0402_1005Metric" (at 389.5852 242.57 0)
-      (effects (font (size 1.27 1.27)) hide)
-    )
-    (property "Datasheet" "~" (at 388.62 238.76 0)
-      (effects (font (size 1.27 1.27)) hide)
-    )
-    (property "LCSC" "C52923" (at 388.62 238.76 0)
-      (effects (font (size 1.27 1.27)) hide)
-    )
-    (property "DNF" "" (at 388.62 238.76 0)
-      (effects (font (size 1.27 1.27)) hide)
-    )
-    (pin "1")
-    (pin "2")
-    (instances
-      (project "sensor-epaper"
-        (path "/8b915f44-d92b-4376-8a4d-f445b50a784a"
-          (reference "C48") (unit 1) (value "1u") (footprint "Capacitor_SMD:C_0402_1005Metric")
-        )
-      )
-    )
-  )
   (symbol (lib_id "Connector:TestPoint") (at 355.6 88.9 90) (unit 1)
     (in_bom yes) (on_board yes) (dnp no)
@@
       (effects (font (size 1.27 1.27)) (justify left))
     )
-    (property "Value" "1u" (at 66.929 64.643 0)
+    (property "Value" "4u7" (at 66.929 64.643 0)
       (effects (font (size 1.27 1.27)) (justify left))
     )
@@
       (effects (font (size 1.27 1.27)) hide)
     )
-    (property "LCSC" "C52923" (at 69.85 63.5 0)
+    (property "LCSC" "C19666" (at 69.85 63.5 0)
       (effects (font (size 1.27 1.27)) hide)
     )
@@
       (project "sensor-epaper"
         (path "/8b915f44-d92b-4376-8a4d-f445b50a784a"
-          (reference "C44") (unit 1) (value "1u") (footprint "Capacitor_SMD:C_0402_1005Metric")
+          (reference "C44") (unit 1) (value "4u7") (footprint "Capacitor_SMD:C_0402_1005Metric")
         )
       )
@@
       (effects (font (size 1.27 1.27)) (justify left))
     )
-    (property "Value" "1u" (at 18.669 64.643 0)
+    (property "Value" "4u7" (at 18.669 64.643 0)
       (effects (font (size 1.27 1.27)) (justify left))
     )
@@
       (effects (font (size 1.27 1.27)) hide)
     )
-    (property "LCSC" "C52923" (at 21.59 63.5 0)
+    (property "LCSC" "C19666" (at 21.59 63.5 0)
       (effects (font (size 1.27 1.27)) hide)
     )
@@
       (project "sensor-epaper"
         (path "/8b915f44-d92b-4376-8a4d-f445b50a784a"
-          (reference "C43") (unit 1) (value "1u") (footprint "Capacitor_SMD:C_0402_1005Metric")
+          (reference "C43") (unit 1) (value "4u7") (footprint "Capacitor_SMD:C_0402_1005Metric")
         )
       )
@@
       (effects (font (size 1.27 1.27)) (justify left))
     )
-    (instances
-      (project "sensor-epaper"
-        (path "/8b915f44-d92b-4376-8a4d-f445b50a784a" (page "2"))
-      )
-    )
   )
   (sheet_instances
-    (path "/" (page "1"))
+    (path "/8b915f44-d92b-4376-8a4d-f445b50a784a" (page "1"))
+    (path "/8b915f44-d92b-4376-8a4d-f445b50a784a/717c6736-2a95-4424-a35e-11020ba9e52f" (page "2"))
   )
 )
